File: SterownikOswietlenia/Eagle/SterownikOswietlenia.sch (EAGLE design)
At the start: 15 parts, among them IC1 MEGA8-AI, T1 BT138-V

Commit message: uporzą▲dkowane opisy elementów
Parts:
- removed C6: 100n, rcl:C-EUC1206
- removed U$2: AK3001-3, RD:AK3001-3
- added C1, C2: 22p, rcl:C-EUC1206
- added D1, D10, D11, D12, D13, D14, D15, D16, D17, D18, D19, D2, D20, D21, D22, D23, D24, D25, D3, D4, D5, D6, D7, D8, D9: 1N4148, diode:DIODE-MINIMELF
- added Q1: 12MHz, special:XTAL/S
- added R10, R11, R12, R13, R14, R15, R16, R17, R18, R19, R20, R21, R22, R23, R24, R25, R26, R27, R29, R8, R9: 100, rcl:R-EU_R1206
- added R28: 10k, rcl:R-EU_R1206
- added R3, R4, R5, R6, R7: 1k, rcl:R-EU_R1206
- added U$1: AK3001-2, RD:AK3001-2
- added X1, X2, X3, X4, X5, X6, X7, X8: (no value), con-ria-59:AKL59-05
- added X10, X11, X12, X13, X14, X15, X16, X17, X18, X19, X20, X21, X22, X23, X24, X25, X26, X27, X28, X29, X30, X31, X32, X33, X34: (no value), con-ria-59:AKL59-02
- added X9: (no value), con-ptr500:AK500/6
- IC1: value MEGA8-AI -> MEGA32-A; device atmel:MEGA8-AI -> atmel:MEGA32-A
- T1: value BT138-V -> BT138-H; device triac:BT138-V -> triac:BT138-H
Connections:
- new net +24V: X1-4.1, X2-4.1, X3-4.1, X4-4.1, X5-4.1, X6-4.1, X7-4.1, X8-4.1, X9-3.KL, X9-4.KL
- new net BTN-H-0: IC1.(ADC1)PA1, R8.1
- new net BTN-H-1: IC1.(ADC3)PA3, R9.1
- new net BTN-H-2: IC1.(ADC5)PA5, R10.1
- new net BTN-H-3: IC1.(ADC7)PA7, R11.1
- new net BTN-H-4: IC1.(TOSC1)PC6, R12.1
- new net BTN-V-0: IC1.(ADC0)PA0, R25.2
- new net BTN-V-1: IC1.(ADC2)PA2, R24.2
- new net BTN-V-2: IC1.(ADC4)PA4, R23.2
- new net BTN-V-3: IC1.(ADC6)PA6, R22.2
- new net BTN-V-4: IC1.(TOSC2)PC7, R21.2
- new net LED-CKO-0: IC1.(RXD)PD0, R13.2
- new net LED-CKO-1: IC1.(TXD)PD1, R14.2
- new net LED-CKO-2: IC1.(INT0)PD2, R15.2
- new net LED-CKO-3: IC1.(INT1)PD3, R16.2
- new net LED-CKO-4: IC1.(OC1B)PD4, R17.2
- new net LED-CKO-5: IC1.(OC1A)PD5, R18.2
- new net LED-CKO-6: IC1.(ICP)PD6, R19.2
- new net LED-CKO-7: IC1.(OC2)PD7, R20.2
- new net LED-SDO: IC1.(TCK)PC2, X1-2.1, X2-2.1, X3-2.1, X4-2.1, X5-2.1, X6-2.1, X7-2.1, X8-2.1
- new net M$44: R12.2, X30-1.1, X31-1.1, X32-1.1, X33-1.1, X34-1.1
- new net N$10: D2.A, X11-2.1
- new net N$113: D10.C, D15.C, D20.C, D25.C, D5.C, R21.1, R7.2
- new net N$12: D3.A, X12-2.1
- new net N$13: D4.A, X13-2.1
- new net N$131: D14.C, D19.C, D24.C, D4.C, D9.C, R22.1, R6.2
- new net N$132: D13.C, D18.C, D23.C, D3.C, D8.C, R23.1, R5.2
- new net N$133: D12.C, D17.C, D2.C, D22.C, D7.C, R24.1, R4.2
- new net N$134: D1.C, D11.C, D16.C, D21.C, D6.C, R25.1, R3.2
- new net N$14: R14.1, X2-1.1
- new net N$15: R15.1, X3-1.1
- new net N$16: R16.1, X4-1.1
- new net N$17: R17.1, X5-1.1
- new net N$18: D5.A, X14-2.1
- new net N$19: D10.A, X19-2.1
- new net N$20: D9.A, X18-2.1
- new net N$21: D8.A, X17-2.1
- new net N$22: D7.A, X16-2.1
- new net N$23: D6.A, X15-2.1
- new net N$24: D11.A, X20-2.1
- new net N$25: D12.A, X21-2.1
- new net N$26: D13.A, X22-2.1
- new net N$27: D14.A, X23-2.1
- new net N$28: D15.A, X24-2.1
- new net N$29: D20.A, X29-2.1
- new net N$30: D19.A, X28-2.1
- new net N$32: D17.A, X26-2.1
- new net N$33: D16.A, X25-2.1
- new net N$34: D21.A, X30-2.1
- new net N$35: D22.A, X31-2.1
- new net N$36: D23.A, X32-2.1
- new net N$37: D24.A, X33-2.1
- new net N$38: D25.A, X34-2.1
- new net N$39: R18.1, X6-1.1
- new net N$40: R8.2, X10-1.1, X11-1.1, X12-1.1, X13-1.1, X14-1.1
- new net N$41: R9.2, X15-1.1, X16-1.1, X17-1.1, X18-1.1, X19-1.1
- new net N$42: R10.2, X20-1.1, X21-1.1, X22-1.1, X23-1.1, X24-1.1
- new net N$43: R11.2, X25-1.1, X26-1.1, X27-1.1, X28-1.1, X29-1.1
- new net N$44: R19.1, X7-1.1
- new net N$45: R20.1, X8-1.1
- new net N$46: C1.1, IC1.XTAL2, Q1.1
- new net N$47: C2.1, IC1.XTAL1, Q1.2
- new net N$49: R27.1, X9-2.KL
- new net N$50: R26.1, X9-1.KL
- new net N$51: IC1.(TDI)PC5, R29.1
- new net N$52: D18.A, X27-2.1
- new net N$7: R13.1, X1-1.1
- new net N$9: D1.A, X10-2.1
- new net POWER-IO-0: IC1.(TDO)PC4, R27.2
- new net TEST_FREQUENCY: IC1.(AIN0/INT2)PB2
- net GND: now also C1.2, C2.2, IC1.GND, IC1.GND1, IC1.GND2, IC1.GND@1, OK1.C, R3.1, R4.1, R5.1, R6.1, R7.1, X1-5.1, X2-5.1, X3-5.1, X4-5.1, X5-5.1, X6-5.1, X7-5.1, X8-5.1, X9-5.KL, X9-6.KL; no longer C6.2, LED1.C
- net I2C-SCL: now also IC1.PC0(SCL); no longer IC1.PC5(ADC5/SCL)
- net I2C-SDA: now also IC1.PC1(SDA); no longer IC1.PC4(ADC4/SDA)
- net ISP-MISO: now also IC1.(MISO)PB6; no longer IC1.PB4(MISO)
- net ISP-MOSI: now also IC1.(MOSI)PB5; no longer IC1.PB3(MOSI/OC2)
- net ISP-SCK: now also IC1.(SCK)PB7; no longer IC1.PB5(SCK)
- net LED-POWER: now also R26.2, R29.2; no longer IC1.PD0(RXD)
- net N$1: now also U$1G$2.KL; no longer U$2G$2.KL
- net N$5: now also LED1.C, OK1.A; no longer LED1.A, OK1.C
- net N$6: now also LED1.A; no longer OK1.A
- net N$8: now also U$1G$1.KL; no longer U$2G$1.KL
- net RESET: now also IC1.RESET, R28.1; no longer IC1.PC6(/RESET)
- net VCC: now also IC1.VCC, IC1.VCC1, IC1.VCC2, R28.2, X1-3.1, X2-3.1, X3-3.1, X4-3.1, X5-3.1, X6-3.1, X7-3.1, X8-3.1; no longer C6.1
Other:
- moved on the sheet: C4, C5, F1, L1, LED1, OK1, PAD1, PAD2, R1, R2, SV2, T1
